File: pcb/qca7000.kicad_sch (KiCad schematic)
At the start: 113 parts, among them J1 Conn_01x20, J2 JTAG, J3 FLASH, U1 AT25SF081-SSHD-X, Y1 25MHz

Commit message: v2, new filter, rbias
Parts:
- removed C57, C58, C59: 10uF 25V, Capacitor_SMD:C_0603_1608Metric, symbol Device:C_Small
- removed D1, D2, D3, D5, D6, D7, D8, D9: 1N4148W, Diode_SMD:D_SOD-123, symbol Diode:1N4148W
- removed D4: 4V7, Diode_SMD:D_SOD-123, symbol Device:D_Zener
- added C8: 1.5nF, Capacitor_SMD:C_0603_1608Metric, symbol Device:C_Small
- added D1, D2, D3, D4: B5819W, Diode_SMD:D_SOD-123, symbol Diode:1N5819
- added D5: 3V9, Diode_SMD:D_SMA, symbol Device:D_Zener
- added D6, D7: BAV99, Package_TO_SOT_SMD:SOT-23, symbol Diode:BAV99
- added L1, L2: 1.8uH, Inductor_SMD:L_0603_1608Metric, symbol Device:L
- C12, C35, C36, C37: value 100nF -> 10uF 10V; LCSC C14663 -> C19702
- C13, C14, C2, C3, C4: value 100nF -> 220pF; LCSC C14663 -> C1603
- C15, C24, C7: value 100nF -> 1.5nF; LCSC C14663 -> C1595
- C41, C42, C52, C53, C54, C55, C56: value 10uF 25V -> 10uF 10V; LCSC C96446 -> C19702
- C51: value 10uF 25V -> 100nF; LCSC C96446 -> C14663
- L11, L8, L9: value Bead 600 -> 1.8uH; LCSC C1002 -> C78153
- L3, L4: value Bead 600 -> 270nH; LCSC C1002 -> C381901
- R1, R2: value R_Small -> 22; LCSC (none) -> C23345
- R15, R17, R20, R22, R4, R8, R9: LCSC (none) -> C25804
- R3, R5: value R_Small -> 2.5k; LCSC (none) -> C304065
- U1: value AT25SF081-SSHD-X -> 25Q16; footprint Package_SO:SOIC-8_3.9x4.9mm_P1.27mm -> Package_SO:SOP-8_5.28x5.23mm_P1.27mm; LCSC (none) -> C115407
- Y1: LCSC C331585 -> C9006
Connections:
- net +1V2_C: now also C52.2, C53.2
- net +3V3_D: now also C35.2, C36.2, C37.2, C41.2, C51.1, L7.2; no longer C37.1, C51.2, C52.2, C53.2
- net GND: now also C10.1, C12.1, C15.1, C24.1, C3.2, C35.1, C36.1, C37.1, C4.1, C51.2, C9.1, D1.2 (A), D2.2 (A), D5.2 (A), D6.1 (K), D7.1 (K), L1.2, L2.1; no longer C3.1, C35.2, C36.2, C37.2, C51.1
- net RXIN_N: now also C13.1, L3.2, L8.1, D7.3 (K); no longer C24.1, L9.2
- net RXIN_P: now also C14.2, L4.2, L9.2, D6.3 (K); no longer C24.2, L11.2
- net RX_N: now also R1.2; no longer R1.1
- net RX_P: now also R2.2; no longer R2.1
- net TXOUT_N: now also C6.1, D1.1 (K), D3.2 (A); no longer C7.1
- net TXOUT_P: now also C5.1, D2.1 (K), D4.2 (A); no longer C4.1
- net TX_N: now also C6.2; no longer C7.2
- net TX_P: now also C5.2; no longer C4.2
- net at C15.2, L11.1: now also C24.2, D6.2 (A), D7.2 (A); no longer L8.2
- net +3V3_A: now reaches C11.1, C33.1, D10.32 (DVDDHLD), D10.36 (XTAL_DVDD), L6.1
- net +3V3_A: now also C12.2, L11.2; no longer C3.2, C35.1, C36.1, C41.2
- new net: C13.2, C14.1, L8.2, L9.1
- new net: C10.2, C9.2, D3.1 (K), D4.1 (K), D5.1 (K), L7.1
- new net: C7.1, L3.1
- new net: C3.1, C7.2, L1.1, R1.1
- new net: C4.2, C8.2, L2.2, R2.1
- new net: C8.1, L4.1
Other:
- note added: "1N5819HW 4pcs"
- note added: "25q16"
- note added: "3rd Order Butterworth Bandpass Lower Cutoff Freq. = 1.900 MHz; Upper Cutoff Freq. = 31.00 MHz https://rf-tools.com/lc-filter/"
- note added: "M25P16"
- moved on the sheet: C11, J2, L6, R15, R17, R18, R20, R22
